File: board/kicad/power.kicad_sch (KiCad schematic)
At the start: 19 parts, among them J1 USB4105-GF-A, J2 Battery 1S Li-ion, U1 USBLC6-2SC6, U2 nPM1300-QEAA-R7

Commit message: Added microphone and battery contacts
Parts:
- removed J2: Battery 1S Li-ion, Connector_JST:JST_SH_SM02B-SRSS-TB_1x02-1MP_P1.00mm_Horizontal, symbol Connector_Generic:Conn_01x02
- added J2, J7: GT-BTP30002-0500B-015A, cmd-z5:BAT-SMD_2P-P3.00_G-Switch_GT-BTP30002-0500B-015A, symbol Connector_Generic_MountingPin:Conn_01x02_MountingPin
Connections:
- net GND: now also J7.1 (Pin_1)
- net VBAT: now also J2.2 (Pin_2)
- net MIC_VDD: now reaches U2.8 (GPIO1)
- no-connect marks 9 -> 12
Other:
- note added: "Battery +"
- note added: "Battery -"
- note added: "Battery contacts: 2x G-Switch side-push springs (one per terminal): + on pin 2, - on pin 1, other pin and fixing foot not connected. Charging is disabled at power-up; firmware must set charge current and VTERM over I2C."
- note removed: "Charging is disabled at power-up; firmware must set charge current and VTERM over I2C."

Commit message: Added extra battery contacts header
Parts:
- added J8: Battery header, Connector_PinHeader_2.54mm:PinHeader_1x02_P2.54mm_Vertical, symbol Connector_Generic:Conn_01x02
Connections:
- net GND: now also J8.2 (Pin_2)
- net VBAT: now also J8.1 (Pin_1)
Other:
- note added: "2.54 mm header, not fitted: 1 = VBAT, 2 = GND"
Changed lines of the file:
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@@
+		)
+	)
+	(symbol
+		(lib_id "Connector_Generic:Conn_01x02")
+		(at 100.33 160.02 0)
+		(unit 1)
+		(exclude_from_sim no)
+		(in_bom yes)
+		(on_board yes)
+		(dnp yes)
+		(property "Reference" "J8"
+			(at 97 154 0)
+			(effects
+				(font
+					(size 1.27 1.27)
+				)
+				(justify left)
+			)
+		)
+		(property "Value" "Battery header"
+			(at 103 158 0)
+			(effects
+				(font
+					(size 1.27 1.27)
+				)
+				(justify left)
+			)
+		)
+		(property "Footprint" "Connector_PinHeader_2.54mm:PinHeader_1x02_P2.54mm_Vertical"
+			(at 100.33 160.02 0)
+			(hide yes)
+			(effects
+				(font
+					(size 1.27 1.27)
+				)
+			)
+		)
+		(property "Datasheet" ""
+			(at 100.33 160.02 0)
+			(hide yes)
+			(effects
+				(font
+					(size 1.27 1.27)
+				)
+			)
+		)
+		(property "Description" "Generic connector, single row, 01x02, script generated (kicad-library-utils/schlib/autogen/connector/)"
+			(at 100.33 160.02 0)
+			(hide yes)
+			(effects
+				(font
+					(size 1.27 1.27)
+				)
+			)
+		)
+		(pin "1"
+		)
+		(pin "2"
+		)
+		(instances
+			(project "cmd-z5"
+				(path "/6abffa09-a441-4dde-b1c7-3053cb1129f2/c246016d-b8d4-41e1-afd7-6e94ddc5dfd4"
+					(reference "J8")
+					(unit 1)
+				)
+			)
+		)
+	)
+	(wire
+		(pts
+			(xy 95.25 160.02)
+			(xy 92.71 160.02)
+		)
+		(stroke
+			(width 0)
+			(type default)
+		)
+	)
+	(symbol
+		(lib_id "cmd-z5:VBAT")
+		(at 92.71 160.02 90)
+		(unit 1)
+		(exclude_from_sim no)
+		(in_bom no)
+		(on_board yes)
+		(dnp no)
+		(property "Reference" "#PWR135"
+			(at 92.71 160.02 90)
+			(hide yes)
+			(effects
+				(font
+					(size 1.27 1.27)
+				)
+			)
+		)
+		(property "Value" "VBAT"
+			(at 87.63 160.02 90)
+			(effects
+				(font
+					(size 1.27 1.27)
+				)
+				(justify left)
+			)
+		)
+		(property "Footprint" ""
+			(at 92.71 160.02 90)
+			(hide yes)
+			(effects
+				(font
+					(size 1.27 1.27)
+				)
+			)
+		)
+		(property "Datasheet" ""
+			(at 92.71 160.02 90)
+			(hide yes)
+			(effects
+				(font
+					(size 1.27 1.27)
+				)
+			)
+		)
+		(property "Description" "Power symbol creates a global label with name \"VBAT\""
+			(at 92.71 160.02 90)
+			(hide yes)
+			(effects
+				(font
+					(size 1.27 1.27)
+				)
+			)
+		)
+		(pin "1"
+		)
+		(instances
+			(project "cmd-z5"
+				(path "/6abffa09-a441-4dde-b1c7-3053cb1129f2/c246016d-b8d4-41e1-afd7-6e94ddc5dfd4"
+					(reference "#PWR135")
+					(unit 1)
+				)
+			)
+		)
+	)
+	(wire
+		(pts
+			(xy 95.25 162.56)
+			(xy 92.71 162.56)
+		)
+		(stroke
+			(width 0)
+			(type default)
+		)
+	)
+	(symbol
+		(lib_id "power:GND")
+		(at 92.71 162.56 270)
+		(unit 1)
+		(exclude_from_sim no)
+		(in_bom no)
+		(on_board yes)
+		(dnp no)
+		(property "Reference" "#PWR136"
+			(at 92.71 162.56 90)
+			(hide yes)
+			(effects
+				(font
+					(size 1.27 1.27)
+				)
+			)
+		)
+		(property "Value" "GND"
+			(at 87.63 162.56 90)
+			(effects
+				(font
+					(size 1.27 1.27)
+				)
+				(justify right)
+			)
+		)
+		(property "Footprint" ""
+			(at 92.71 162.56 90)
+			(hide yes)
+			(effects
+				(font
+					(size 1.27 1.27)
+				)
+			)
+		)
+		(property "Datasheet" ""
+			(at 92.71 162.56 90)
+			(hide yes)
+			(effects
+				(font
+					(size 1.27 1.27)
+				)
+			)
+		)
+		(property "Description" "Power symbol creates a global label with name \"GND\" , ground"
+			(at 92.71 162.56 90)
+			(hide yes)
+			(effects
+				(font
+					(size 1.27 1.27)
+				)
+			)
+		)
+		(pin "1"
+		)
+		(instances
+			(project "cmd-z5"
+				(path "/6abffa09-a441-4dde-b1c7-3053cb1129f2/c246016d-b8d4-41e1-afd7-6e94ddc5dfd4"
+					(reference "#PWR136")
+					(unit 1)
+				)
+			)
+		)
+	)
+	(text "2.54 mm header, not fitted:\n1 = VBAT, 2 = GND"
+		(exclude_from_sim no)
+		(at 85 168 0)
+		(effects
+			(font
+				(size 1.27 1.27)
+			)
+			(justify left top)
 		)
 	)
