File: board/kicad/ui.kicad_sch (KiCad schematic)
At the start: 25 parts, among them J5 X05A20H26G, J6 FH12-28S-0.5SH(55), Q1 DMG1024UV, Q2 DMG1016UDW, U7 PAM8302AASCR

Commit message: Replaced FFC connectors with low profile ones
Parts:
- J5: value X05A20H26G -> KH-FPC0.5-H1.0SMT-26P-QCHF; footprint Connector_FFC-FPC:Hirose_FH12-26S-0.5SH_1x26-1MP_P0.50mm_Horizontal -> cmd-z5:FPC-SMD_26P-P0.50_KH-FPC0.5-H1.0SMT-26P-QCHF; LCSC C528050 -> C3250122; Note Footprint placeholder: create X05A20H26G footprint -> (none)
- J6: value FH12-28S-0.5SH(55) -> KH-FPC0.5-H1.0SMT-28P-QCHF; footprint Connector_FFC-FPC:Hirose_FH12-28S-0.5SH_1x28-1MP_P0.50mm_Horizontal -> cmd-z5:FPC-SMD_28P-P0.50_KH-FPC0.5-H1.0SMT-28P-QCHF; LCSC C597983 -> C3250123
Changed lines of the file:
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@@
 			)
 		)
-		(property "Value" "X05A20H26G"
+		(property "Value" "KH-FPC0.5-H1.0SMT-26P-QCHF"
 			(at 36.83 127 0)
 			(effects
@@
 			)
 		)
-		(property "Footprint" "Connector_FFC-FPC:Hirose_FH12-26S-0.5SH_1x26-1MP_P0.50mm_Horizontal"
+		(property "Footprint" "cmd-z5:FPC-SMD_26P-P0.50_KH-FPC0.5-H1.0SMT-26P-QCHF"
 			(at 39.37 85.09 0)
 			(hide yes)
@@
 			)
 		)
-		(property "LCSC" "C528050"
-			(at 39.37 85.09 0)
-			(hide yes)
-			(effects
-				(font
-					(size 1.27 1.27)
-				)
-			)
-		)
-		(property "Note" "Footprint placeholder: create X05A20H26G footprint"
+		(property "LCSC" "C3250122"
 			(at 39.37 85.09 0)
 			(hide yes)
@@
 			)
 		)
-		(property "Value" "FH12-28S-0.5SH(55)"
+		(property "Value" "KH-FPC0.5-H1.0SMT-28P-QCHF"
 			(at 177.8 129.54 0)
 			(effects
@@
 			)
 		)
-		(property "Footprint" "Connector_FFC-FPC:Hirose_FH12-28S-0.5SH_1x28-1MP_P0.50mm_Horizontal"
+		(property "Footprint" "cmd-z5:FPC-SMD_28P-P0.50_KH-FPC0.5-H1.0SMT-28P-QCHF"
 			(at 180.34 85.09 0)
 			(hide yes)
@@
 			)
 		)
-		(property "LCSC" "C597983"
+		(property "LCSC" "C3250123"
 			(at 180.34 85.09 0)
 			(hide yes)

Commit message: Fixed component positions
Parts:
- added D4, D5, D6, D7: green, LED_SMD:LED_0603_1608Metric, symbol Device:LED
- added R27, R28, R29, R30: 330, Resistor_SMD:R_0402_1005Metric, symbol Device:R_Small
Connections:
- net LED_K_SW: now also R27.2, R28.2, R29.2, R30.2
- net VSYS: now also D4.2 (A), D5.2 (A), D6.2 (A), D7.2 (A)
- new net: D5.1 (K), R28.1
- new net: D7.1 (K), R30.1
- new net: D6.1 (K), R29.1
- new net: D4.1 (K), R27.1
Other:
- note added: "0603 green, 330R each: ~3 mA (3.6 V) to ~7 mA (5 V USB). On with the flex LEDs (Q1A, LED_EN)."
- note added: "Board LEDs"
