File: board/kicad/cmd-z5.kicad_pcb (KiCad board)
At the start: 2 copper layers, 43 x 82.4 mm, 120 parts, among them J1 USB4105-GF-A, J2 GT-BTP30002-0500B-015A, J3 SWD, J4 TBS M10N, J5 KH-FPC0.5-H1.0SMT-26P-QCHF, J6 KH-FPC0.5-H1.0SMT-28P-QCHF, J7 GT-BTP30002-0500B-015A, J8 Battery header, Q1 DMG1024UV, Q2 DMG1016UDW, U1 USBLC6-2SC6, U2 nPM1300-QEAA-R7, U3 nRF52840-QIAA-R, U4 LIS2DH12TR, U5 Wio-SX1262, U6 TPS610997YFFR, U7 PAM8302AASCR, U8 TLV9001IDCKR, Y1 32 MHz CL=10pF, Y2 32.768 kHz CL=7pF

Commit message: Optimized placement
Parts:
- U6: footprint Package_BGA:Texas_DSBGA-6_0.855x1.255mm_Layout2x3_P0.4mm_LevelB -> cmd-z5:Texas_DSBGA-6_0.855x1.255mm_Layout2x3_P0.4mm_LevelB
- Y2: footprint Crystal:Crystal_SMD_2012-2Pin_2.0x1.2mm -> cmd-z5:Crystal_SMD_2012-2Pin_2.0x1.2mm
- moved R9 37.9 mm to (92.2, 87.5)
- moved R17 30.2 mm to (99.9, 98.4), turned to 90 degrees
- moved R12 27.6 mm to (99.9, 93.4)
- moved Q2 27.0 mm to (102.0, 97.4), turned to 180 degrees
- moved R15 25.9 mm to (100.3, 94.8), turned to -90 degrees
- moved Q1 24.3 mm to (102.2, 93.8), turned to 180 degrees
- moved R16 23.7 mm to (103.9, 96.8), turned to 90 degrees
- moved D2 23.5 mm to (95.6, 93.0), turned to 90 degrees
- moved R13 22.4 mm to (101.8, 91.9)
- moved R14 22.2 mm to (103.9, 93.2)
- moved D3 21.7 mm to (105.4, 97.5)
- moved D1 21.2 mm to (92.4, 93.1)
- moved C45 14.7 mm to (123.8, 108.2), turned to 0 degrees
- moved C22 14.1 mm to (92.2, 86.2), turned to 180 degrees
- moved C25 13.4 mm to (105.9, 86.0), turned to -90 degrees
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Other:
- copper layers 2 -> 6
