File: board/kicad/cmd-z5.kicad_pcb (KiCad board)
At the start: 6 copper layers, 43 x 82.4 mm, 120 parts, among them J1 USB4105-GF-A, J2 GT-BTP30002-0500B-015A, J3 SWD, J4 TBS M10N, J5 KH-FPC0.5-H1.0SMT-26P-QCHF, J6 KH-FPC0.5-H1.0SMT-28P-QCHF, J7 GT-BTP30002-0500B-015A, J8 Battery header, Q1 DMG1024UV, Q2 DMG1016UDW, U1 USBLC6-2SC6, U2 nPM1300-QEAA-R7, U3 nRF52840-QIAA-R, U4 LIS2DH12TR, U5 Wio-SX1262, U6 TPS610997YFFR, U7 PAM8302AASCR, U8 TLV9001IDCKR, Y1 32 MHz CL=10pF, Y2 32.768 kHz CL=7pF

Commit message: Started some manual routing
Routing:
- net LORA_MISO: track 0.00 -> 41.4 mm, vias 0 -> 2
- net LORA_MOSI: track 0.00 -> 39.9 mm, vias 0 -> 2
- net LORA_SCK: track 0.00 -> 38.7 mm, vias 0 -> 2
- net LORA_NSS: track 0.00 -> 34.1 mm, vias 0 -> 2
- net LCD_D0: track 0.00 -> 29.0 mm, vias 0 -> 1
- net LCD_D1: track 0.00 -> 28.7 mm, vias 0 -> 1
- net LCD_D2: track 0.00 -> 27.8 mm, vias 0 -> 1
- net LCD_D3: track 0.00 -> 27.4 mm, vias 0 -> 1
- net LCD_D4: track 0.00 -> 27.2 mm, vias 0 -> 1
- net LORA_DIO1: track 0.00 -> 26.8 mm, vias 0 -> 1
- net LCD_D5: track 0.00 -> 26.6 mm, vias 0 -> 1
- net LCD_A0: track 0.00 -> 26.5 mm, vias 0 -> 1
- net LORA_BUSY: track 0.00 -> 26.1 mm, vias 0 -> 1
- net LCD_D6: track 0.00 -> 24.8 mm, vias 0 -> 1
- net LID_SW: track 0.00 -> 23.8 mm, vias 0 -> 2
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- added copper zone on In3.Cu, net +3V0
- added copper zone on In1.Cu, net GND
- added copper zone on In4.Cu, net GND
