File: board/kicad/radio_gps.kicad_sch (KiCad schematic)
At the start: 15 parts, among them J4 TBS M10N, U5 Wio-SX1262, U6 TPS610997YFFR

Commit message: Added board outline and did initial component placement
Parts:
- AE2: footprint (none) -> RF_Antenna:Texas_SWRA416_868MHz_915MHz
- U5: footprint (none) -> cmd-z5:Seeed_Wio-SX1262
Other:
- note added: "Meshtastic: SX126X_RXEN = RF_SW, DIO2 as RF switch, TCXO 1.8 V on DIO3."
- note removed: "Meshtastic: SX126X_RXEN = RF_SW, DIO2 as RF switch, TCXO 1.8 V on DIO3. Footprint: create from datasheet."
Changed lines of the file:
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@@
 			)
 		)
-		(property "Footprint" ""
+		(property "Footprint" "cmd-z5:Seeed_Wio-SX1262"
 			(at 80.01 64.77 0)
 			(hide yes)
@@
 			)
 		)
-		(property "Footprint" ""
+		(property "Footprint" "RF_Antenna:Texas_SWRA416_868MHz_915MHz"
 			(at 165.1 44.45 0)
 			(hide yes)
@@
 		)
 	)
-	(text "Meshtastic: SX126X_RXEN = RF_SW, DIO2 as RF switch,\nTCXO 1.8 V on DIO3. Footprint: create from datasheet."
+	(text "Meshtastic: SX126X_RXEN = RF_SW, DIO2 as RF switch,\nTCXO 1.8 V on DIO3."
 		(exclude_from_sim no)
 		(at 100 105 0)

Commit message: Few physical modifications
Parts:
- AE2: footprint RF_Antenna:Texas_SWRA416_868MHz_915MHz -> cmd-z5:Texas_SWRA416_868MHz_915MHz_Mirrored
- J4: footprint Connector_JST:JST_SH_SM04B-SRSS-TB_1x04-1MP_P1.00mm_Horizontal -> cmd-z5:SolderPads_1x04_P2.00mm_SMD
Changed lines of the file:
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@@
 			)
 		)
-		(property "Footprint" "RF_Antenna:Texas_SWRA416_868MHz_915MHz"
+		(property "Footprint" "cmd-z5:Texas_SWRA416_868MHz_915MHz_Mirrored"
 			(at 165.1 44.45 0)
 			(hide yes)
@@
 			)
 		)
-		(property "Footprint" "Connector_JST:JST_SH_SM04B-SRSS-TB_1x04-1MP_P1.00mm_Horizontal"
+		(property "Footprint" "cmd-z5:SolderPads_1x04_P2.00mm_SMD"
 			(at 149.86 180.34 0)
 			(hide yes)

Commit message: Optimized placement
Parts:
- U6: footprint Package_BGA:Texas_DSBGA-6_0.855x1.255mm_Layout2x3_P0.4mm_LevelB -> cmd-z5:Texas_DSBGA-6_0.855x1.255mm_Layout2x3_P0.4mm_LevelB
Changed lines of the file:
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@@
 			)
 		)
-		(property "Footprint" "Package_BGA:Texas_DSBGA-6_0.855x1.255mm_Layout2x3_P0.4mm_LevelB"
+		(property "Footprint" "cmd-z5:Texas_DSBGA-6_0.855x1.255mm_Layout2x3_P0.4mm_LevelB"
 			(at 59.69 180.34 0)
 			(hide yes)
